Commit message: ferdig for dagen

File: urdf/robotarm.urdf.xacro (robot description, xacro)
@@ -1,12 +1,25 @@
 <?xml version="1.0"?>
-<robot name="macroed" xmlns:xacro="http://ros.org/wiki/xacro">
+<robot name="yes" xmlns:xacro="http://ros.org/wiki/xacro">
   <material name="blue">
      <color rgba="0 0 0.8 1"/>
   </material>
+<!-- -->
+<!-- Base dimensions -->
 <xacro:property name="basex" value="0.2" />
 <xacro:property name="basey" value="0.2" />
 <xacro:property name="basez" value="0.05" />
+<!-- Turntable dimensions -->
 <xacro:property name="turntable_height" value="0.01" />
 <xacro:property name="turntable_radius" value="0.09" />
+<!-- Motor dimensions -->
+<xacro:property name="motorx" value="0.0356" />
+<xacro:property name="motory" value="0.0355" />
+<xacro:property name="motorz" value="0.0506" />
+<!-- Mounting plate dimensions -->
+<xacro:property name="mpx" value="0.0356" />
+<xacro:property name="mpy" value="0.0355" />
+<xacro:property name="mpz" value="0.0206" />
+<xacro:property name="girder_len" value="0.0635" />
+<!-- Base -->
 <link name="base_link">
   <visual>
@@ -21,5 +34,5 @@
       <cylinder radius = "${turntable_radius}" length = "${turntable_height}"/>
     </geometry>
-    <origin xyz ="0 0 ${(basez+turntable_height)/10}"/>
+    <origin xyz ="0 0 ${(basez+turntable_height)/2}"/>
     <material name="blue"/>
   </visual>
@@ -28,6 +41,55 @@
   <parent link="base_link"/>
   <child link="turntable"/>
-  <origin xyz="0 0 ${basez/2}"/>
+  <origin xyz="0 0 0"/>
   <axis xyz ="0 0 1"/>
 </joint>
+<xacro:macro name="motor" params="prefix z_coord parent">
+<link name="${prefix}_motor">
+  <visual>
+    <geometry>
+      <box size ="${motorx} ${motory} ${motorz}"/>
+    </geometry>
+    <origin xyz ="0 0 ${z_coord}"/>
+    <material name="blue"/>
+  </visual>
+</link>
+<joint name="${parent}_to_${prefix}_motor" type="fixed">
+  <parent link="${parent}"/>
+  <child link="${prefix}_motor"/>
+  <origin xyz="0 0 0"/>
+  <axis xyz ="1 0 0"/>
+</joint>
+</xacro:macro>
+<xacro:macro name="mounting_plate" params="prefix z_coord parent">
+<link name="${prefix}_mounting_plate">
+  <visual>
+    <geometry>
+      <box size ="${mpx} ${mpy} ${mpz}"/>
+    </geometry>
+    <origin xyz ="0 0 ${z_coord}"/>
+  </visual>
+</link>
+<joint name="${parent}_to_${prefix}_mounting_plate" type="continuous">
+  <parent link="${parent}"/>
+  <child link="${prefix}_mounting_plate"/>
+  <origin xyz="0 0 ${motorz}"/>
+  <axis xyz ="1 0 0"/>
+</joint>
+</xacro:macro>
+<xacro:motor prefix="second" z_coord="${basez+turntable_height}" parent="turntable"/>
+<xacro:mounting_plate prefix="first" z_coord="${turntable_height+motorz}" parent="second_motor"/>
+<link name="girder">
+  <visual>
+    <geometry>
+      <box size ="${mpx} ${mpy} ${girder_len}"/>
+    </geometry>
+    <origin xyz ="0 0 ${mpz/2}"/>
+      <material name="blue"/>
+  </visual>
+</link>
+<joint name="first_mounting_plate_to_girder" type="continuous">
+  <parent link="first_mounting_plate"/>
+  <child link="girder"/>
+  <axis xyz ="1 0 0"/>
+</joint>
 </robot>

Commit message: added som extra joints

File: urdf/robotarm.urdf.xacro (robot description, xacro)
@@ -3,4 +3,7 @@
   <material name="blue">
      <color rgba="0 0 0.8 1"/>
+  </material>
+  <material name="cyan">
+     <color rgba="0 1 1 1"/>
   </material>
 <!-- -->
@@ -34,5 +37,5 @@
       <cylinder radius = "${turntable_radius}" length = "${turntable_height}"/>
     </geometry>
-    <origin xyz ="0 0 ${(basez+turntable_height)/2}"/>
+    <origin xyz ="0 0 0"/>
     <material name="blue"/>
   </visual>
@@ -41,5 +44,5 @@
   <parent link="base_link"/>
   <child link="turntable"/>
-  <origin xyz="0 0 0"/>
+  <origin xyz="0 0 ${(basez+turntable_height)/2}"/>
   <axis xyz ="0 0 1"/>
 </joint>
@@ -50,5 +53,5 @@
       <box size ="${motorx} ${motory} ${motorz}"/>
     </geometry>
-    <origin xyz ="0 0 ${z_coord}"/>
+    <origin xyz ="0 0 ${motorz/2}"/>
     <material name="blue"/>
   </visual>
@@ -57,5 +60,5 @@
   <parent link="${parent}"/>
   <child link="${prefix}_motor"/>
-  <origin xyz="0 0 0"/>
+  <origin xyz="0 0 ${z_coord}"/>
   <axis xyz ="1 0 0"/>
 </joint>
@@ -67,5 +70,5 @@
       <box size ="${mpx} ${mpy} ${mpz}"/>
     </geometry>
-    <origin xyz ="0 0 ${z_coord}"/>
+    <origin xyz ="0 0 ${mpz/2}"/>
   </visual>
 </link>
@@ -73,10 +76,10 @@
   <parent link="${parent}"/>
   <child link="${prefix}_mounting_plate"/>
-  <origin xyz="0 0 ${motorz}"/>
+  <origin xyz="0 0 ${z_coord}"/>
   <axis xyz ="1 0 0"/>
 </joint>
 </xacro:macro>
-<xacro:motor prefix="second" z_coord="${basez+turntable_height}" parent="turntable"/>
-<xacro:mounting_plate prefix="first" z_coord="${turntable_height+motorz}" parent="second_motor"/>
+<xacro:motor prefix="second" z_coord="${turntable_height/2}" parent="turntable"/>
+<xacro:mounting_plate prefix="first" z_coord="${motorz}" parent="second_motor"/>
 <link name="girder">
   <visual>
@@ -84,12 +87,17 @@
       <box size ="${mpx} ${mpy} ${girder_len}"/>
     </geometry>
-    <origin xyz ="0 0 ${mpz/2}"/>
-      <material name="blue"/>
+    <origin xyz ="0 0 ${girder_len/2}"/>
+      <material name="cyan"/>
   </visual>
 </link>
-<joint name="first_mounting_plate_to_girder" type="continuous">
+<joint name="first_mounting_plate_to_girder" type="fixed">
   <parent link="first_mounting_plate"/>
   <child link="girder"/>
+  <origin xyz="0 0 ${mpz}"/>
   <axis xyz ="1 0 0"/>
 </joint>
+<xacro:motor prefix="third" z_coord="${girder_len}" parent="girder"/>
+<xacro:mounting_plate prefix="second" z_coord="${motorz}" parent="third_motor"/>
+<xacro:motor prefix="fourth" z_coord="${mpz}" parent="second_mounting_plate"/>
+<xacro:mounting_plate prefix="third" z_coord="${motorz}" parent="fourth_motor"/>
 </robot>

Commit message: ferdig med visuals for robotarm

File: urdf/robotarm.urdf.xacro (robot description, xacro)
@@ -31,4 +31,9 @@
     </geometry>
   </visual>
+  <collision>
+  <geometry>
+    <cylinder length="0.6" radius="0.2"/>
+  </geometry>
+</collision>
 </link>
 <link name="turntable">
@@ -85,4 +90,5 @@
   <visual>
     <geometry>
+      <!--<mesh filename="package://five_dof_robotarm/stl_files/25Girder.igs"/>-->
       <box size ="${mpx} ${mpy} ${girder_len}"/>
     </geometry>
@@ -101,3 +107,56 @@
 <xacro:motor prefix="fourth" z_coord="${mpz}" parent="second_mounting_plate"/>
 <xacro:mounting_plate prefix="third" z_coord="${motorz}" parent="fourth_motor"/>
+<!-- Wrist rotate kit -->
+<link name="wrist_rk">
+  <visual>
+    <geometry>
+      <box size ="${mpx} ${mpy} ${motorz}"/>
+    </geometry>
+    <origin xyz ="0 0 ${motorz/2}"/>
+      <material name="cyan"/>
+  </visual>
+</link>
+<joint name="third_mounting_plate_to_wrist_rk" type="fixed">
+  <parent link="third_mounting_plate"/>
+  <child link="wrist_rk"/>
+  <origin xyz="0 0 ${mpz}"/>
+  <axis xyz ="0 0 1"/>
+</joint>
+<!-- Wrist -->
+<link name="wrist">
+  <visual>
+    <geometry>
+      <box size ="${mpx} ${mpy*2} ${motorz/2}"/>
+    </geometry>
+    <origin xyz ="0 0 ${motorz/4}"/>
+      <material name="blue"/>
+  </visual>
+</link>
+<joint name="wrist_rk_to_wrist" type="continuous">
+  <parent link="wrist_rk"/>
+  <child link="wrist"/>
+  <origin xyz="0 0 ${motorz}"/>
+  <axis xyz ="0 0 1"/>
+</joint>
+<!-- Gripper-->
+<xacro:property name="finger_length" value="0.1" />
+<xacro:property name="finger_width" value="0.0356" />
+<xacro:macro name="finger" params="prefix invert">
+<link name="${prefix}_finger">
+  <visual>
+    <geometry>
+      <box size ="${finger_width} ${finger_width/4} ${finger_length}"/>
+    </geometry>
+    <origin xyz ="0 0 ${finger_length/2}"/>
+  </visual>
+</link>
+<joint name="$wrist_to_${prefix}_finger" type="continuous">
+  <parent link="wrist"/>
+  <child link="${prefix}_finger"/>
+  <origin xyz="0 ${invert*mpy} 0"/>
+  <axis xyz ="${invert} 0 0"/>
+</joint>
+</xacro:macro>
+<xacro:finger prefix="right" invert="1"/>
+<xacro:finger prefix="left" invert="-1"/>
 </robot>

Commit message: Dagens arbeid

File: urdf/robotarm.urdf.xacro (robot description, xacro)
@@ -1,10 +1,8 @@
 <?xml version="1.0"?>
 <robot name="yes" xmlns:xacro="http://ros.org/wiki/xacro">
-  <material name="blue">
-     <color rgba="0 0 0.8 1"/>
-  </material>
-  <material name="cyan">
-     <color rgba="0 1 1 1"/>
-  </material>
+<xacro:include filename="$(find five_dof_robotarm)/urdf/materials.xacro" />
+<material name="cyan">
+   <color rgba="0 1 1 1"/>
+</material>
 <!-- -->
 <!-- Base dimensions -->
@@ -24,4 +22,12 @@
 <xacro:property name="mpz" value="0.0206" />
 <xacro:property name="girder_len" value="0.0635" />
+<!-- Mass -->
+<xacro:property name="mass_motor" value="0.126"/>
+<!-- Fixing robot to Gazebo base_link -->
+<link name="world"/>
+  <joint name="fixed" type="fixed">
+    <parent link="world"/>
+    <child link="base_link"/>
+  </joint>
 <!-- Base -->
 <link name="base_link">
@@ -33,5 +39,5 @@
   <collision>
   <geometry>
-    <cylinder length="0.6" radius="0.2"/>
+    <box size ="${basex} ${basey} ${basez}"/>
   </geometry>
 </collision>
@@ -43,5 +49,5 @@
     </geometry>
     <origin xyz ="0 0 0"/>
-    <material name="blue"/>
+    <material name="orange"/>
   </visual>
 </link>
@@ -68,4 +74,13 @@
   <axis xyz ="1 0 0"/>
 </joint>
+<inertial>
+   <origin xyz="0 0 ${height1/2}" rpy="0 0 0"/>
+   <mass value="${mass_motor}"/>
+   <inertia
+   ixx="${mass / 12.0 * (width*width + height1*height1)}" ixy="0.0" ixz="0.0"
+   iyy="${mass / 12.0 * (height1*height1 + width*width)}" iyz="0.0"
+   izz="${mass / 12.0 * (width*width + width*width)}"/>
+ </inertial>
+</link>
 </xacro:macro>
 <xacro:macro name="mounting_plate" params="prefix z_coord parent">
@@ -155,4 +170,5 @@
   <child link="${prefix}_finger"/>
   <origin xyz="0 ${invert*mpy} 0"/>
+   <limit effort="1000.0" lower="0.0" upper="${0.548*invert}" velocity="0.5"/>
   <axis xyz ="${invert} 0 0"/>
 </joint>

Commit message: spisepause

File: urdf/robotarm.urdf.xacro (robot description, xacro)
@@ -24,5 +24,6 @@
 <!-- Mass -->
 <xacro:property name="mass_motor" value="0.126"/>
-<!-- Fixing robot to Gazebo base_link -->
+<xacro:property name="mass_mp" value="0.01"/> <!--Mass mounting plate-->
+<!-- Fixing robot to Gazebo base_link-->
 <link name="world"/>
   <joint name="fixed" type="fixed">
@@ -36,4 +37,5 @@
       <box size ="${basex} ${basey} ${basez}"/>
     </geometry>
+    <origin xyz="0 0 0" rpy="0 0 0"/>
   </visual>
   <collision>
@@ -42,4 +44,9 @@
   </geometry>
 </collision>
+<inertial>
+  <origin xyz="0 0 0" rpy="0 0 0"/>
+  <mass value="2"/>
+  <inertia ixx="1" ixy="0" ixz="0" iyy="1" iyz="0" izz="1" />
+</inertial>
 </link>
 <link name="turntable">
@@ -58,4 +65,5 @@
   <axis xyz ="0 0 1"/>
 </joint>
+<!--Motor macro-->
 <xacro:macro name="motor" params="prefix z_coord parent">
 <link name="${prefix}_motor">
@@ -67,4 +75,18 @@
     <material name="blue"/>
   </visual>
+<collision>
+  <origin xyz ="0 0 ${motorz/2}"/>
+  <geometry>
+    <box size ="${motorx} ${motory} ${motorz}"/>
+  </geometry>
+</collision>
+<inertial>
+   <origin xyz="0 0 ${motorz/2}" rpy="0 0 0"/>
+   <mass value="${mass_motor}"/>
+   <inertia
+   ixx="${mass_motor / 12.0 * (motorx*motorx + motorz*motorz)}" ixy="0.0" ixz="0.0"
+   iyy="${mass_motor / 12.0 * (motorz*motorz + motory*motory)}" iyz="0.0"
+   izz="${mass_motor / 12.0 * (motorx*motorx + motory*motory)}"/>
+ </inertial>
 </link>
 <joint name="${parent}_to_${prefix}_motor" type="fixed">
@@ -74,14 +96,6 @@
   <axis xyz ="1 0 0"/>
 </joint>
-<inertial>
-   <origin xyz="0 0 ${height1/2}" rpy="0 0 0"/>
-   <mass value="${mass_motor}"/>
-   <inertia
-   ixx="${mass / 12.0 * (width*width + height1*height1)}" ixy="0.0" ixz="0.0"
-   iyy="${mass / 12.0 * (height1*height1 + width*width)}" iyz="0.0"
-   izz="${mass / 12.0 * (width*width + width*width)}"/>
- </inertial>
-</link>
 </xacro:macro>
+<!--Mounting plate macro-->
 <xacro:macro name="mounting_plate" params="prefix z_coord parent">
 <link name="${prefix}_mounting_plate">
@@ -90,6 +104,20 @@
       <box size ="${mpx} ${mpy} ${mpz}"/>
     </geometry>
-    <origin xyz ="0 0 ${mpz/2}"/>
-  </visual>
+    <origin xyz ="0 0 ${mpz/2}" rpy="0 0 0"/>
+  </visual>
+<collision>
+  <origin xyz ="0 0 ${mpz/2}"/>
+  <geometry>
+    <box size ="${mpx} ${mpy} ${mpz}"/>
+  </geometry>
+</collision>
+<inertial>
+   <origin xyz="0 0 ${mpz/2}" rpy="0 0 0"/>
+   <mass value="${mass_mp}"/>
+   <inertia
+   ixx="${mass_mp / 12.0 * (mpx*mpx + mpz*mpz)}" ixy="0.0" ixz="0.0"
+   iyy="${mass_mp / 12.0 * (mpz*mpz + mpy*mpy)}" iyz="0.0"
+   izz="${mass_mp / 12.0 * (mpx*mpx + mpy*mpy)}"/>
+ </inertial>
 </link>
 <joint name="${parent}_to_${prefix}_mounting_plate" type="continuous">
@@ -98,4 +126,5 @@
   <origin xyz="0 0 ${z_coord}"/>
   <axis xyz ="1 0 0"/>
+  <dynamics damping="0.01"/>
 </joint>
 </xacro:macro>
@@ -111,4 +140,18 @@
       <material name="cyan"/>
   </visual>
+  <collision>
+    <origin xyz ="0 0 ${girder_len/2}"/>
+    <geometry>
+      <box size ="${mpx} ${mpy} ${girder_len}"/>
+    </geometry>
+  </collision>
+  <inertial>
+     <origin xyz="0 0 ${girder_len/2}" rpy="0 0 0"/>
+     <mass value="${mass_mp*3}"/>
+     <inertia
+     ixx="${mass_mp*3 / 12.0 * (mpx*mpx + girder_len*girder_len)}" ixy="0.0" ixz="0.0"
+     iyy="${mass_mp*3 / 12.0 * (girder_len*girder_len + mpy*mpy)}" iyz="0.0"
+     izz="${mass_mp*3 / 12.0 * (mpx*mpx + mpy*mpy)}"/>
+   </inertial>
 </link>
 <joint name="first_mounting_plate_to_girder" type="fixed">
@@ -131,4 +174,18 @@
       <material name="cyan"/>
   </visual>
+  <collision>
+    <origin xyz ="0 0 ${motorz/2}"/>
+    <geometry>
+      <box size ="${mpx} ${mpy} ${motorz}"/>
+    </geometry>
+  </collision>
+  <inertial>
+     <origin xyz="0 0 ${motorz/2}" rpy="0 0 0"/>
+     <mass value="${mass_motor}"/>
+     <inertia
+     ixx="${mass_motor / 12.0 * (motorx*motorx + motorz*motorz)}" ixy="0.0" ixz="0.0"
+     iyy="${mass_motor / 12.0 * (motorz*motorz + motory*motory)}" iyz="0.0"
+     izz="${mass_motor / 12.0 * (motorx*motorx + motory*motory)}"/>
+   </inertial>
 </link>
 <joint name="third_mounting_plate_to_wrist_rk" type="fixed">
@@ -147,4 +204,18 @@
       <material name="blue"/>
   </visual>
+  <collision>
+    <origin xyz ="0 0 ${motorz/4}"/>
+    <geometry>
+      <box size ="${mpx} ${mpy*2} ${motorz/2}"/>
+    </geometry>
+  </collision>
+  <inertial>
+     <origin xyz="0 0 ${motorz/4}" rpy="0 0 0"/>
+     <mass value="${mass_motor}"/>
+     <inertia
+     ixx="${mass_motor / 12.0 * (motorx*motorx + motorz*motorz/4)}" ixy="0.0" ixz="0.0"
+     iyy="${mass_motor / 12.0 * (motorz*motorz/4 + motory*motory*4)}" iyz="0.0"
+     izz="${mass_motor / 12.0 * (motorx*motorx + motory*motory*4)}"/>
+   </inertial>
 </link>
 <joint name="wrist_rk_to_wrist" type="continuous">
@@ -155,6 +226,7 @@
 </joint>
 <!-- Gripper-->
-<xacro:property name="finger_length" value="0.1" />
+<xacro:property name="finger_length" value="0.08" />
 <xacro:property name="finger_width" value="0.0356" />
+<xacro:property name="mass_finger" value="0.01" />
 <xacro:macro name="finger" params="prefix invert">
 <link name="${prefix}_finger">
@@ -165,11 +237,26 @@
     <origin xyz ="0 0 ${finger_length/2}"/>
   </visual>
+  <collision>
+    <origin xyz ="0 0 ${finger_length/2}"/>
+    <geometry>
+      <box size ="${finger_width} ${finger_width/4} ${finger_length}"/>
+    </geometry>
+  </collision>
+  <inertial>
+     <origin xyz="0 0 ${finger_length/2}" rpy="0 0 0"/>
+     <mass value="${mass_finger}"/>
+     <inertia
+     ixx="${mass_finger / 12.0 * (finger_width*finger_width + finger_length*finger_length)}" ixy="0.0" ixz="0.0"
+     iyy="${mass_finger / 12.0 * (finger_length*finger_length + finger_width*finger_width/16)}" iyz="0.0"
+     izz="${mass_finger / 12.0 * (finger_width*finger_width + finger_width*finger_width/16)}"/>
+   </inertial>
 </link>
 <joint name="$wrist_to_${prefix}_finger" type="continuous">
   <parent link="wrist"/>
   <child link="${prefix}_finger"/>
-  <origin xyz="0 ${invert*mpy} 0"/>
+  <origin xyz="0 ${invert*mpy} ${mpz}"/>
    <limit effort="1000.0" lower="0.0" upper="${0.548*invert}" velocity="0.5"/>
   <axis xyz ="${invert} 0 0"/>
+  <dynamics damping="0.01"/>
 </joint>
 </xacro:macro>

Commit message: Bra dag

File: urdf/robotarm.urdf.xacro (robot description, xacro)
@@ -4,10 +4,10 @@
 <!-- -->
 <!-- Base dimensions -->
-<xacro:property name="basex" value="0.2" />
-<xacro:property name="basey" value="0.2" />
-<xacro:property name="basez" value="0.05" />
+<xacro:property name="basex" value="0.1143" />
+<xacro:property name="basey" value="0.1143" />
+<xacro:property name="basez" value="0.0381" />
 <!-- Turntable dimensions -->
 <xacro:property name="turntable_height" value="0.01" />
-<xacro:property name="turntable_radius" value="0.09" />
+<xacro:property name="turntable_radius" value="0.055" />
 <!-- Motor dimensions -->
 <xacro:property name="motorx" value="0.0356" />
@@ -22,4 +22,5 @@
 <xacro:property name="mass_motor" value="0.126"/>
 <xacro:property name="mass_mp" value="0.01"/> <!--Mass mounting plate-->
+<xacro:property name="mass_tt" value="0.05"/> <!--Turntable-->
 <!-- Operating limits(ol) [rad]-->
 <xacro:property name="motor_ol" value="1.92"/><!--110deg-->
@@ -63,4 +64,18 @@
     <material name="orange"/>
   </visual>
+  <collision>
+    <origin xyz ="0 0 0"/>
+    <geometry>
+      <cylinder radius= "${turntable_radius}" length= "${turntable_height}"/>
+    </geometry>
+  </collision>
+  <inertial>
+     <origin xyz="0 0 0" rpy="0 0 0"/>
+     <mass value="${mass_tt}"/>
+     <inertia
+       ixx="${mass_tt / 12.0 * (3*turntable_radius*turntable_radius + turntable_height*turntable_height)}" ixy="0.0" ixz="0.0"
+       iyy="${mass_tt / 12.0 * (3*turntable_radius*turntable_radius + turntable_height*turntable_height)}" iyz="0.0"
+       izz="${mass_tt / 12.0 * (turntable_radius*turntable_radius)}"/>
+   </inertial>
 </link>
 <joint name="base_to_turntable" type="continuous">
@@ -70,4 +85,13 @@
   <axis xyz ="0 0 1"/>
 </joint>
+<transmission name="turntable_trans">
+  <type>transmisson_interface/SimpleTransmission</type>
+  <actuator name="$turntable_motor">
+    <mechanicalReduction>1</mechanicalReduction>
+  </actuator>
+  <joint name="base_to_turntable">
+    <hardwareInterface>PositionJointInterface</hardwareInterface>
+  </joint>
+</transmission>
 <!--Motor macro-->
 <xacro:macro name="motor" params="prefix z_coord parent">
@@ -149,5 +173,5 @@
     <origin xyz ="0 0 ${girder_len/2}"/>
     <geometry>
-      <box size ="${mpx} ${mpy} ${mpz}"/>
+      <box size ="${mpx} ${mpy} ${girder_len}"/>
     </geometry>
   </collision>

Commit message: One step closer

File: urdf/robotarm.urdf.xacro (robot description, xacro)
@@ -39,9 +39,4 @@
     <origin xyz="0 0 0" rpy="0 0 0"/>
   </visual>
-  <collision>
-  <geometry>
-    <box size ="${basex} ${basey} ${basez}"/>
-  </geometry>
-</collision>
 <inertial>
   <origin xyz="0 0 0" rpy="0 0 0"/>
@@ -91,5 +86,5 @@
   </actuator>
   <joint name="base_to_turntable">
-    <hardwareInterface>PositionJointInterface</hardwareInterface>
+    <hardwareInterface>hardware_interface/EffortJointInterface</hardwareInterface>
   </joint>
 </transmission>
@@ -295,5 +290,5 @@
 <gazebo>
    <plugin name="gazebo_ros_control" filename="libgazebo_ros_control.so">
-     <robotNamespace>/</robotNamespace>
+     <robotNamespace>/five_dof_robotarm</robotNamespace>
    </plugin>
  </gazebo>
