Commit message: The arm is now steerable from Python!

File: urdf/simp_inert.urdf.xacro (robot description, xacro)
@@ -1,6 +1,9 @@
 <?xml version="1.0"?>
-<robot name="five_dof_robotarm" xmlns:xacro="http://ros.org/wiki/xacro">
+<robot name="yes" xmlns:xacro="http://ros.org/wiki/xacro">
 <xacro:include filename="$(find five_dof_robotarm)/urdf/materials.xacro" />
-<!-- -->
+<!--
+Gazebo wont accept macroed values on the inertia section, so I have replaced all
+the equations with one in the start just so it will work.
+ -->
 <!-- Base dimensions -->
 <xacro:property name="basex" value="0.1143" />
@@ -25,5 +28,5 @@
 <!-- Operating limits(ol) [rad]-->
 <xacro:property name="motor_ol" value="1.92"/><!--110deg-->
-<!-- Fixing robot to world frame
+<!-- Fixing robot to world frame-->
 <link name="world"/>
   <joint name="fixed" type="fixed">
@@ -31,5 +34,4 @@
     <child link="base_link"/>
   </joint>
--->
 <!-- Base -->
 <link name="base_link">
@@ -69,8 +71,5 @@
      <origin xyz="0 0 0" rpy="0 0 0"/>
      <mass value="${mass_tt}"/>
-     <inertia
-       ixx="${mass_tt / 12.0 * (3*turntable_radius*turntable_radius + turntable_height*turntable_height)}" ixy="0.0" ixz="0.0"
-       iyy="${mass_tt / 12.0 * (3*turntable_radius*turntable_radius + turntable_height*turntable_height)}" iyz="0.0"
-       izz="${mass_tt / 12.0 * (turntable_radius*turntable_radius)}"/>
+     <inertia ixx="1" ixy="0" ixz="0" iyy="1" iyz="0" izz="1" />
    </inertial>
 </link>
@@ -109,8 +108,5 @@
    <origin xyz="0 0 ${motorz/2}" rpy="0 0 0"/>
    <mass value="${mass_motor}"/>
-   <inertia
-   ixx="${mass_motor / 12.0 * (motorx*motorx + motorz*motorz)}" ixy="0.0" ixz="0.0"
-   iyy="${mass_motor / 12.0 * (motorz*motorz + motory*motory)}" iyz="0.0"
-   izz="${mass_motor / 12.0 * (motorx*motorx + motory*motory)}"/>
+   <inertia ixx="1" ixy="0" ixz="0" iyy="1" iyz="0" izz="1" />
  </inertial>
 </link>
@@ -140,8 +136,5 @@
    <origin xyz="0 0 ${mpz/2}" rpy="0 0 0"/>
    <mass value="${mass_mp}"/>
-   <inertia
-   ixx="${mass_mp / 12.0 * (mpx*mpx + mpz*mpz)}" ixy="0.0" ixz="0.0"
-   iyy="${mass_mp / 12.0 * (mpz*mpz + mpy*mpy)}" iyz="0.0"
-   izz="${mass_mp / 12.0 * (mpx*mpx + mpy*mpy)}"/>
+   <inertia ixx="1" ixy="0" ixz="0" iyy="1" iyz="0" izz="1" />
  </inertial>
 </link>
@@ -154,4 +147,13 @@
   <limit effort="10" lower="${-motor_ol}" upper="${motor_ol}" velocity="5"/>
 </joint>
+<transmission name="turntable_trans">
+  <type>transmisson_interface/SimpleTransmission</type>
+  <actuator name="${prefix}_arm_motor">
+    <mechanicalReduction>1</mechanicalReduction>
+  </actuator>
+  <joint name="${parent}_to_${prefix}_mounting_plate">
+    <hardwareInterface>hardware_interface/EffortJointInterface</hardwareInterface>
+  </joint>
+</transmission>
 </xacro:macro>
 <xacro:motor prefix="second" z_coord="${turntable_height/2}" parent="turntable"/>
@@ -175,8 +177,5 @@
      <origin xyz="0 0 ${girder_len/2}" rpy="0 0 0"/>
      <mass value="${mass_mp*3}"/>
-     <inertia
-     ixx="${mass_mp*3 / 12.0 * (mpx*mpx + girder_len*girder_len)}" ixy="0.0" ixz="0.0"
-     iyy="${mass_mp*3 / 12.0 * (girder_len*girder_len + mpy*mpy)}" iyz="0.0"
-     izz="${mass_mp*3 / 12.0 * (mpx*mpx + mpy*mpy)}"/>
+     <inertia ixx="1" ixy="0" ixz="0" iyy="1" iyz="0" izz="1" />
    </inertial>
 </link>
@@ -209,8 +208,5 @@
      <origin xyz="0 0 ${motorz/2}" rpy="0 0 0"/>
      <mass value="${mass_motor}"/>
-     <inertia
-     ixx="${mass_motor / 12.0 * (motorx*motorx + motorz*motorz)}" ixy="0.0" ixz="0.0"
-     iyy="${mass_motor / 12.0 * (motorz*motorz + motory*motory)}" iyz="0.0"
-     izz="${mass_motor / 12.0 * (motorx*motorx + motory*motory)}"/>
+     <inertia ixx="1" ixy="0" ixz="0" iyy="1" iyz="0" izz="1" />
    </inertial>
 </link>
@@ -239,8 +235,5 @@
      <origin xyz="0 0 ${motorz/4}" rpy="0 0 0"/>
      <mass value="${mass_motor}"/>
-     <inertia
-     ixx="${mass_motor / 12.0 * (motorx*motorx + motorz*motorz/4)}" ixy="0.0" ixz="0.0"
-     iyy="${mass_motor / 12.0 * (motorz*motorz/4 + motory*motory*4)}" iyz="0.0"
-     izz="${mass_motor / 12.0 * (motorx*motorx + motory*motory*4)}"/>
+     <inertia ixx="1" ixy="0" ixz="0" iyy="1" iyz="0" izz="1" />
    </inertial>
 </link>
@@ -272,8 +265,5 @@
      <origin xyz="0 0 ${finger_length/2}" rpy="0 0 0"/>
      <mass value="${mass_finger}"/>
-     <inertia
-     ixx="${mass_finger / 12.0 * (finger_width*finger_width + finger_length*finger_length)}" ixy="0.0" ixz="0.0"
-     iyy="${mass_finger / 12.0 * (finger_length*finger_length + finger_width*finger_width/16)}" iyz="0.0"
-     izz="${mass_finger / 12.0 * (finger_width*finger_width + finger_width*finger_width/16)}"/>
+     <inertia ixx="1" ixy="0" ixz="0" iyy="1" iyz="0" izz="1" />
    </inertial>
 </link>

Commit message: Added more joint control(Fikk jobb i dag, så det er litt vanskelig å konsentrere

File: urdf/simp_inert.urdf.xacro (robot description, xacro)
@@ -80,13 +80,4 @@
   <axis xyz ="0 0 1"/>
 </joint>
-<transmission name="turntable_trans">
-  <type>transmisson_interface/SimpleTransmission</type>
-  <actuator name="$turntable_motor">
-    <mechanicalReduction>1</mechanicalReduction>
-  </actuator>
-  <joint name="base_to_turntable">
-    <hardwareInterface>hardware_interface/EffortJointInterface</hardwareInterface>
-  </joint>
-</transmission>
 <!--Motor macro-->
 <xacro:macro name="motor" params="prefix z_coord parent">
@@ -147,13 +138,4 @@
   <limit effort="10" lower="${-motor_ol}" upper="${motor_ol}" velocity="5"/>
 </joint>
-<transmission name="turntable_trans">
-  <type>transmisson_interface/SimpleTransmission</type>
-  <actuator name="${prefix}_arm_motor">
-    <mechanicalReduction>1</mechanicalReduction>
-  </actuator>
-  <joint name="${parent}_to_${prefix}_mounting_plate">
-    <hardwareInterface>hardware_interface/EffortJointInterface</hardwareInterface>
-  </joint>
-</transmission>
 </xacro:macro>
 <xacro:motor prefix="second" z_coord="${turntable_height/2}" parent="turntable"/>
@@ -278,4 +260,35 @@
 <xacro:finger prefix="right" invert="1"/>
 <xacro:finger prefix="left" invert="-1"/>
+<!-- Control -->
+<!-- First link control-->
+<transmission name="turntable_trans">
+  <type>transmisson_interface/SimpleTransmission</type>
+  <actuator name="$turntable_motor">
+    <mechanicalReduction>1</mechanicalReduction>
+  </actuator>
+  <joint name="base_to_turntable">
+    <hardwareInterface>hardware_interface/EffortJointInterface</hardwareInterface>
+  </joint>
+</transmission>
+<!-- Second link control -->
+<transmission name="joint2">
+  <type>transmisson_interface/SimpleTransmission</type>
+  <actuator name="joint2_motor">
+    <mechanicalReduction>1</mechanicalReduction>
+  </actuator>
+  <joint name="second_motor_to_first_mounting_plate">
+    <hardwareInterface>hardware_interface/EffortJointInterface</hardwareInterface>
+  </joint>
+</transmission>
+<!-- Third link control -->
+<transmission name="joint3">
+  <type>transmisson_interface/SimpleTransmission</type>
+  <actuator name="joint3_motor">
+    <mechanicalReduction>1</mechanicalReduction>
+  </actuator>
+  <joint name="third_motor_to_second_mounting_plate">
+    <hardwareInterface>hardware_interface/EffortJointInterface</hardwareInterface>
+  </joint>
+</transmission>
 <!-- Gazebo plugin for ROS Control -->
 <gazebo>

Commit message: Tweaks and control

File: urdf/simp_inert.urdf.xacro (robot description, xacro)
@@ -99,5 +99,7 @@
    <origin xyz="0 0 ${motorz/2}" rpy="0 0 0"/>
    <mass value="${mass_motor}"/>
-   <inertia ixx="1" ixy="0" ixz="0" iyy="1" iyz="0" izz="1" />
+   <inertia ixx="0.1" ixy="0" ixz="0"
+            iyy="0.1" iyz="0"
+            izz="0.1" />
  </inertial>
 </link>
@@ -127,5 +129,7 @@
    <origin xyz="0 0 ${mpz/2}" rpy="0 0 0"/>
    <mass value="${mass_mp}"/>
-   <inertia ixx="1" ixy="0" ixz="0" iyy="1" iyz="0" izz="1" />
+   <inertia ixx="0.1" ixy="0" ixz="0"
+            iyy="0.1" iyz="0"
+            izz="0.1" />
  </inertial>
 </link>
@@ -135,8 +139,9 @@
   <origin xyz="0 0 ${z_coord}"/>
   <axis xyz ="1 0 0"/>
-  <dynamics damping="0.1"/>
-  <limit effort="10" lower="${-motor_ol}" upper="${motor_ol}" velocity="5"/>
+  <dynamics damping="1"/>
+  <limit effort="10" lower="${-motor_ol}" upper="${motor_ol}" velocity="50"/>
 </joint>
 </xacro:macro>
+<!-- Second joint -->
 <xacro:motor prefix="second" z_coord="${turntable_height/2}" parent="turntable"/>
 <xacro:mounting_plate prefix="first" z_coord="${motorz}" parent="second_motor"/>
@@ -169,6 +174,8 @@
 </joint>
 <xacro:motor prefix="third" z_coord="${girder_len}" parent="girder"/>
+<!-- Third joint  -->
 <xacro:mounting_plate prefix="second" z_coord="${motorz}" parent="third_motor"/>
 <xacro:motor prefix="fourth" z_coord="${mpz}" parent="second_mounting_plate"/>
+<!-- Fourth joint -->
 <xacro:mounting_plate prefix="third" z_coord="${motorz}" parent="fourth_motor"/>
 <!-- Wrist rotate kit -->
@@ -199,5 +206,5 @@
   <axis xyz ="0 0 1"/>
 </joint>
-<!-- Wrist -->
+<!-- Fifth joint  (Wrist) -->
 <link name="wrist">
   <visual>
@@ -250,5 +257,5 @@
    </inertial>
 </link>
-<joint name="$wrist_to_${prefix}_finger" type="revolute">
+<joint name="$wrist_to_${prefix}_finger" type="fixed">
   <parent link="wrist"/>
   <child link="${prefix}_finger"/>
@@ -260,5 +267,5 @@
 <xacro:finger prefix="right" invert="1"/>
 <xacro:finger prefix="left" invert="-1"/>
-<!-- Control -->
+<!--Control -->
 <!-- First link control-->
 <transmission name="turntable_trans">
@@ -266,4 +273,5 @@
   <actuator name="$turntable_motor">
     <mechanicalReduction>1</mechanicalReduction>
+    <motorTorqueConstant>100</motorTorqueConstant>
   </actuator>
   <joint name="base_to_turntable">
@@ -275,5 +283,5 @@
   <type>transmisson_interface/SimpleTransmission</type>
   <actuator name="joint2_motor">
-    <mechanicalReduction>1</mechanicalReduction>
+  <!--mechanicalReduction>1</mechanicalReduction-->
   </actuator>
   <joint name="second_motor_to_first_mounting_plate">
@@ -285,7 +293,17 @@
   <type>transmisson_interface/SimpleTransmission</type>
   <actuator name="joint3_motor">
-    <mechanicalReduction>1</mechanicalReduction>
+    <!--mechanicalReduction>1</mechanicalReduction-->
   </actuator>
   <joint name="third_motor_to_second_mounting_plate">
+    <hardwareInterface>hardware_interface/EffortJointInterface</hardwareInterface>
+  </joint>
+</transmission>
+<!-- Fourth link control -->
+<transmission name="joint4">
+  <type>transmisson_interface/SimpleTransmission</type>
+  <actuator name="joint4_motor">
+    <!--mechanicalReduction>1</mechanicalReduction-->
+  </actuator>
+  <joint name="fourth_motor_to_third_mounting_plate">
     <hardwareInterface>hardware_interface/EffortJointInterface</hardwareInterface>
   </joint>

Commit message: Two way communication with Gazebo has been established. Fixed more realistic inertias

File: urdf/simp_inert.urdf.xacro (robot description, xacro)
@@ -71,5 +71,5 @@
      <origin xyz="0 0 0" rpy="0 0 0"/>
      <mass value="${mass_tt}"/>
-     <inertia ixx="1" ixy="0" ixz="0" iyy="1" iyz="0" izz="1" />
+     <inertia ixx="0.0082" ixy="0" ixz="0" iyy="0.0082" iyz="0" izz="0.0076" />
    </inertial>
 </link>
@@ -99,7 +99,7 @@
    <origin xyz="0 0 ${motorz/2}" rpy="0 0 0"/>
    <mass value="${mass_motor}"/>
-   <inertia ixx="0.1" ixy="0" ixz="0"
-            iyy="0.1" iyz="0"
-            izz="0.1" />
+   <inertia ixx="0.004" ixy="0" ixz="0"
+            iyy="0.004" iyz="0"
+            izz="0.00456" />
  </inertial>
 </link>
@@ -129,7 +129,7 @@
    <origin xyz="0 0 ${mpz/2}" rpy="0 0 0"/>
    <mass value="${mass_mp}"/>
-   <inertia ixx="0.1" ixy="0" ixz="0"
-            iyy="0.1" iyz="0"
-            izz="0.1" />
+   <inertia ixx="0.00014" ixy="0" ixz="0"
+            iyy="0.00014" iyz="0"
+            izz="0.00021" />
  </inertial>
 </link>
@@ -146,4 +146,5 @@
 <xacro:motor prefix="second" z_coord="${turntable_height/2}" parent="turntable"/>
 <xacro:mounting_plate prefix="first" z_coord="${motorz}" parent="second_motor"/>
+<!-- Girder -->
 <link name="girder">
   <visual>
@@ -164,5 +165,5 @@
      <origin xyz="0 0 ${girder_len/2}" rpy="0 0 0"/>
      <mass value="${mass_mp*3}"/>
-     <inertia ixx="1" ixy="0" ixz="0" iyy="1" iyz="0" izz="1" />
+     <inertia ixx="0.00176" ixy="0" ixz="0" iyy="0.00176" iyz="0" izz="0.000842" />
    </inertial>
 </link>
@@ -197,5 +198,7 @@
      <origin xyz="0 0 ${motorz/2}" rpy="0 0 0"/>
      <mass value="${mass_motor}"/>
-     <inertia ixx="1" ixy="0" ixz="0" iyy="1" iyz="0" izz="1" />
+     <inertia ixx="0.004" ixy="0" ixz="0"
+              iyy="0.004" iyz="0"
+              izz="0.00456" />
    </inertial>
 </link>
@@ -206,5 +209,5 @@
   <axis xyz ="0 0 1"/>
 </joint>
-<!-- Fifth joint  (Wrist) -->
+<!-- Fifth joint  (Wrist)-->
 <link name="wrist">
   <visual>
@@ -225,4 +228,6 @@
      <mass value="${mass_motor}"/>
      <inertia ixx="1" ixy="0" ixz="0" iyy="1" iyz="0" izz="1" />
+     <!--<inertia ixx="0.0000473" ixy="0" ixz="0" iyy="0.0000158" iyz="0" izz="0.0000131" />
+   -->
    </inertial>
 </link>
@@ -254,5 +259,5 @@
      <origin xyz="0 0 ${finger_length/2}" rpy="0 0 0"/>
      <mass value="${mass_finger}"/>
-     <inertia ixx="1" ixy="0" ixz="0" iyy="1" iyz="0" izz="1" />
+     <inertia ixx="0.0000001" ixy="0" ixz="0" iyy="0.0000001" iyz="0" izz="0.0000001" />
    </inertial>
 </link>
@@ -306,4 +311,14 @@
   </actuator>
   <joint name="fourth_motor_to_third_mounting_plate">
+    <hardwareInterface>hardware_interface/EffortJointInterface</hardwareInterface>
+  </joint>
+</transmission>
+<!-- Fifth link control -->
+<transmission name="joint5">
+  <type>transmisson_interface/SimpleTransmission</type>
+  <actuator name="joint5_motor">
+    <!--mechanicalReduction>1</mechanicalReduction-->
+  </actuator>
+  <joint name="wrist_rk_to_wrist">
     <hardwareInterface>hardware_interface/EffortJointInterface</hardwareInterface>
   </joint>

Commit message: Fully functional controller

File: urdf/simp_inert.urdf.xacro (robot description, xacro)
@@ -5,5 +5,5 @@
 Gazebo wont accept macroed values on the inertia section, so I have replaced all
 the equations with one in the start just so it will work. Multiplied each value of
-the inertias with 100. Gazebo would go wild if the inertias were too low.
+the inertias with 1000. Gazebo would go wild if the inertias were too low.
  -->
 <!-- Base dimensions -->
@@ -72,5 +72,5 @@
      <origin xyz="0 0 0" rpy="0 0 0"/>
      <mass value="${mass_tt}"/>
-     <inertia ixx="0.0082" ixy="0" ixz="0" iyy="0.0082" iyz="0" izz="0.0076" />
+     <inertia ixx="0.082" ixy="0" ixz="0" iyy="0.082" iyz="0" izz="0.076" />
    </inertial>
 </link>
@@ -100,7 +100,7 @@
    <origin xyz="0 0 ${motorz/2}" rpy="0 0 0"/>
    <mass value="${mass_motor}"/>
-   <inertia ixx="0.004" ixy="0" ixz="0"
-            iyy="0.004" iyz="0"
-            izz="0.00456" />
+   <inertia ixx="0.04" ixy="0" ixz="0"
+            iyy="0.04" iyz="0"
+            izz="0.0456" />
  </inertial>
 </link>
@@ -130,7 +130,7 @@
    <origin xyz="0 0 ${mpz/2}" rpy="0 0 0"/>
    <mass value="${mass_mp}"/>
-   <inertia ixx="0.00014" ixy="0" ixz="0"
-            iyy="0.00014" iyz="0"
-            izz="0.00021" />
+   <inertia ixx="0.0014" ixy="0" ixz="0"
+            iyy="0.0014" iyz="0"
+            izz="0.0021" />
  </inertial>
 </link>
@@ -166,5 +166,5 @@
      <origin xyz="0 0 ${girder_len/2}" rpy="0 0 0"/>
      <mass value="${mass_mp*3}"/>
-     <inertia ixx="0.00176" ixy="0" ixz="0" iyy="0.00176" iyz="0" izz="0.000842" />
+     <inertia ixx="0.0176" ixy="0" ixz="0" iyy="0.0176" iyz="0" izz="0.00842" />
    </inertial>
 </link>
@@ -199,7 +199,7 @@
      <origin xyz="0 0 ${motorz/2}" rpy="0 0 0"/>
      <mass value="${mass_motor}"/>
-     <inertia ixx="0.004" ixy="0" ixz="0"
-              iyy="0.004" iyz="0"
-              izz="0.00456" />
+     <inertia ixx="0.04" ixy="0" ixz="0"
+              iyy="0.04" iyz="0"
+              izz="0.0456" />
    </inertial>
 </link>
@@ -228,7 +228,6 @@
      <origin xyz="0 0 ${motorz/4}" rpy="0 0 0"/>
      <mass value="${mass_motor}"/>
-     <inertia ixx="1" ixy="0" ixz="0" iyy="1" iyz="0" izz="1" />
-     <!--<inertia ixx="0.0000473" ixy="0" ixz="0" iyy="0.0000158" iyz="0" izz="0.0000131" />
-   -->
+     <!--inertia ixx="1" ixy="0" ixz="0" iyy="1" iyz="0" izz="1" /-->
+     <inertia ixx="0.0473" ixy="0" ixz="0" iyy="0.0158" iyz="0" izz="0.0131" />
    </inertial>
 </link>

Commit message: kinematics

File: urdf/simp_inert.urdf.xacro (robot description, xacro)
@@ -30,5 +30,7 @@
 <xacro:property name="motor_ol" value="1.92"/><!--110deg-->
 <!-- Fixing robot to world frame-->
-<link name="world"/>
+<link name="world">
+  <origin xyz="0 0 -100" rpy="0 0 0"/>
+</link>
   <joint name="fixed" type="fixed">
     <parent link="world"/>

Commit message: Inverse Kinematics inc

File: urdf/simp_inert.urdf.xacro (robot description, xacro)
@@ -115,5 +115,5 @@
 </xacro:macro>
 <!--Mounting plate macro-->
-<xacro:macro name="mounting_plate" params="prefix z_coord parent">
+<xacro:macro name="mounting_plate" params="prefix z_coord parent angle">
 <link name="${prefix}_mounting_plate">
   <visual>
@@ -140,5 +140,5 @@
   <parent link="${parent}"/>
   <child link="${prefix}_mounting_plate"/>
-  <origin xyz="0 0 ${z_coord}"/>
+  <origin xyz="0 0 ${z_coord}" rpy="${angle} 0 0" />
   <axis xyz ="1 0 0"/>
   <dynamics damping="1"/>
@@ -148,5 +148,5 @@
 <!-- Second joint -->
 <xacro:motor prefix="second" z_coord="${turntable_height/2}" parent="turntable"/>
-<xacro:mounting_plate prefix="first" z_coord="${motorz}" parent="second_motor"/>
+<xacro:mounting_plate prefix="first" z_coord="${motorz}" parent="second_motor" angle="0"/>
 <!-- Girder -->
 <link name="girder">
@@ -179,8 +179,8 @@
 <xacro:motor prefix="third" z_coord="${girder_len}" parent="girder"/>
 <!-- Third joint  -->
-<xacro:mounting_plate prefix="second" z_coord="${motorz}" parent="third_motor"/>
+<xacro:mounting_plate prefix="second" z_coord="${motorz}" parent="third_motor" angle="0"/>
 <xacro:motor prefix="fourth" z_coord="${mpz}" parent="second_mounting_plate"/>
 <!-- Fourth joint -->
-<xacro:mounting_plate prefix="third" z_coord="${motorz}" parent="fourth_motor"/>
+<xacro:mounting_plate prefix="third" z_coord="${motorz}" parent="fourth_motor" angle="0"/>
 <!-- Wrist rotate kit -->
 <link name="wrist_rk">
@@ -264,5 +264,5 @@
    </inertial>
 </link>
-<joint name="$wrist_to_${prefix}_finger" type="fixed">
+<joint name="wrist_to_${prefix}_finger" type="fixed">
   <parent link="wrist"/>
   <child link="${prefix}_finger"/>

Commit message: Fixed IK solver

File: urdf/simp_inert.urdf.xacro (robot description, xacro)
@@ -28,5 +28,5 @@
 <xacro:property name="mass_tt" value="0.05"/> <!--Turntable-->
 <!-- Operating limits(ol) [rad]-->
-<xacro:property name="motor_ol" value="1.92"/><!--110deg-->
+<xacro:property name="motor_ol" value="3.92"/><!--110deg 1.92 rad-->
 <!-- Fixing robot to world frame-->
 <link name="world">

Commit message: Small update

File: urdf/simp_inert.urdf.xacro (robot description, xacro)
@@ -33,8 +33,4 @@
   <origin xyz="0 0 -100" rpy="0 0 0"/>
 </link>
-  <joint name="fixed" type="fixed">
-    <parent link="world"/>
-    <child link="base_link"/>
-  </joint>
 <!-- Base -->
 <link name="base_link">
@@ -57,4 +53,8 @@
 </collision>
 </link>
+<joint name="fixed" type="fixed">
+  <parent link="world"/>
+  <child link="base_link"/>
+</joint>
 <link name="turntable">
   <visual>
@@ -239,4 +239,5 @@
   <origin xyz="0 0 ${motorz}"/>
   <axis xyz ="0 0 1"/>
+  <limit effort="10" lower="${-motor_ol}" upper="${motor_ol}" velocity="50"/>
 </joint>
 <!-- Gripper-->

Commit message: Matlab Plotting

File: urdf/simp_inert.urdf.xacro (robot description, xacro)
@@ -74,5 +74,5 @@
      <origin xyz="0 0 0" rpy="0 0 0"/>
      <mass value="${mass_tt}"/>
-     <inertia ixx="0.082" ixy="0" ixz="0" iyy="0.082" iyz="0" izz="0.076" />
+     <inertia ixx="0.0082" ixy="0" ixz="0" iyy="0.0082" iyz="0" izz="0.0076" />
    </inertial>
 </link>
@@ -102,7 +102,7 @@
    <origin xyz="0 0 ${motorz/2}" rpy="0 0 0"/>
    <mass value="${mass_motor}"/>
-   <inertia ixx="0.04" ixy="0" ixz="0"
-            iyy="0.04" iyz="0"
-            izz="0.0456" />
+   <inertia ixx="0.004" ixy="0" ixz="0"
+            iyy="0.004" iyz="0"
+            izz="0.00456" />
  </inertial>
 </link>
@@ -132,7 +132,7 @@
    <origin xyz="0 0 ${mpz/2}" rpy="0 0 0"/>
    <mass value="${mass_mp}"/>
-   <inertia ixx="0.0014" ixy="0" ixz="0"
-            iyy="0.0014" iyz="0"
-            izz="0.0021" />
+   <inertia ixx="0.00014" ixy="0" ixz="0"
+            iyy="0.00014" iyz="0"
+            izz="0.00021" />
  </inertial>
 </link>
@@ -168,5 +168,5 @@
      <origin xyz="0 0 ${girder_len/2}" rpy="0 0 0"/>
      <mass value="${mass_mp*3}"/>
-     <inertia ixx="0.0176" ixy="0" ixz="0" iyy="0.0176" iyz="0" izz="0.00842" />
+     <inertia ixx="0.00176" ixy="0" ixz="0" iyy="0.00176" iyz="0" izz="0.000842" />
    </inertial>
 </link>
@@ -201,7 +201,7 @@
      <origin xyz="0 0 ${motorz/2}" rpy="0 0 0"/>
      <mass value="${mass_motor}"/>
-     <inertia ixx="0.04" ixy="0" ixz="0"
-              iyy="0.04" iyz="0"
-              izz="0.0456" />
+     <inertia ixx="0.004" ixy="0" ixz="0"
+              iyy="0.004" iyz="0"
+              izz="0.00456" />
    </inertial>
 </link>
@@ -231,5 +231,5 @@
      <mass value="${mass_motor}"/>
      <!--inertia ixx="1" ixy="0" ixz="0" iyy="1" iyz="0" izz="1" /-->
-     <inertia ixx="0.0473" ixy="0" ixz="0" iyy="0.0158" iyz="0" izz="0.0131" />
+     <inertia ixx="0.00473" ixy="0" ixz="0" iyy="0.00158" iyz="0" izz="0.00131" />
    </inertial>
 </link>
@@ -280,6 +280,6 @@
   <type>transmisson_interface/SimpleTransmission</type>
   <actuator name="$turntable_motor">
-    <mechanicalReduction>1</mechanicalReduction>
-    <motorTorqueConstant>1000</motorTorqueConstant>
+    <!--mechanicalReduction>1</mechanicalReduction-->
+    <!--motorTorqueConstant>1000</motorTorqueConstant-->
   </actuator>
   <joint name="base_to_turntable">
